File: CARP.kicad_pcb (KiCad board)
At the start: 4 copper layers, 95 parts, among them J1 USB_C_Receptacle_USB2.0_14P, J2 Conn_01x10, J3 Conn_01x10, J4 U.fl, SW1 SW_Push, SW2 SW_Push, U1 W25Q128JVSIMTR (16MB), U2 W25Q32RVXHJQ (2MB), U3 LM1117IMPX-3.3, U4 RP2350_60QFN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

Commit message: Preliminary CC1200 decoupling design
Parts:
- moved C26 88.1 mm to (581.5, 145.7), turned to -90 degrees
- moved R16 85.4 mm to (577.7, 153.8)
- moved C42 78.1 mm to (571.7, 147.3), turned to 180 degrees
- moved C41 72.9 mm to (571.7, 149.3), turned to 180 degrees
- moved C40 69.2 mm to (575.7, 153.8), turned to -90 degrees
- moved U7 66.4 mm to (577.0, 149.0)
- moved C43 65.7 mm to (600.5, 153.9)
- moved C44 65.7 mm to (619.6, 153.9)
- moved C45 65.7 mm to (632.3, 166.6)
- moved C50 65.7 mm to (665.3, 141.2)
- moved L4 65.7 mm to (610.7, 153.9)
- moved L5 65.7 mm to (611.9, 166.6)
- moved L8 65.7 mm to (666.5, 155.2)
- moved L9 65.7 mm to (674.2, 155.2)
- moved C46 65.7 mm to (645.0, 141.2)
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Routing:
- net +3.3VA: track 0.00 -> 21.2 mm
- net /GPIO23: track 0.00 -> 4.13 mm
- net /GPIO24: track 0.00 -> 3.93 mm
- net /GPIO21: track 0.00 -> 3.85 mm
- net /CC1200/TCXO_CLK: track 0.00 -> 3.07 mm
- net Net-(U7-LPF1): track 0.00 -> 3.00 mm
- net Net-(U7-LPF0): track 0.00 -> 2.77 mm
- net Net-(U7-DCPL): track 0.00 -> 2.56 mm
- net Net-(U7-DCPL_XOSC): track 0.00 -> 2.40 mm
- net Net-(U7-DCPL_VCO): track 0.00 -> 2.13 mm
- net Net-(U7-DCPL_PFD_CHP): track 0.00 -> 2.02 mm
- net Net-(U7-RBIAS): track 0.00 -> 1.83 mm
Other:
- board text added: "Change 3.3VA traces that are next to eachother with copper pours Probably below RF section replace 3.3V layer with 3.3VA? Rethink components names silkscreen sizes, because they be pretty larg for this scale"
