File: CARP.kicad_pcb (KiCad board)
At the start: 4 copper layers, 95 parts, among them J1 USB_C_Receptacle_USB2.0_14P, J2 Conn_01x10, J3 Conn_01x10, J4 U.fl, SW1 SW_Push, SW2 SW_Push, U1 W25Q128JVSIMTR (16MB), U2 W25Q32RVXHJQ (2MB), U3 LM1117IMPX-3.3, U4 RP2350_60QFN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

Commit message: work
Parts:
- C23: footprint Capacitor_SMD:C_0402_1005Metric -> Capacitor_SMD:C_0603_1608Metric
- JP1: moved to B.Cu
- R14, R15: footprint PCM_Resistor_SMD_AKL:R_0603_1608Metric -> Resistor_SMD:R_0402_1005Metric
- SW2: footprint Button_Switch_SMD:SW_SPST_PTS645Sx43SMTR92 -> Button_Switch_SMD:SW_Push_1P1T_NO_Vertical_Wuerth_434133025816
- moved C3 386.2 mm to (260.5, -86.7), turned to 0 degrees
- moved J3 233.0 mm to (245.7, -32.9)
- moved J2 226.4 mm to (245.9, -38.4), turned to 180 degrees
- moved C25 205.1 mm to (236.2, 204.1)
- moved C24 190.8 mm to (235.4, 196.8), turned to -90 degrees
- moved C2 175.6 mm to (247.2, 209.2), turned to 0 degrees
- moved U5 173.0 mm to (236.5, 201.7), turned to -90 degrees
- moved C1 171.3 mm to (244.8, 209.2), turned to 180 degrees
- moved Y1 158.0 mm to (246.0, 211.9), turned to 0 degrees
- moved R8 143.6 mm to (246.7, 207.6)
- moved R15 143.4 mm to (235.8, 198.2)
- moved C21 138.1 mm to (235.8, 199.2)
- moved U3 136.8 mm to (260.2, 173.7)
- moved R14 136.7 mm to (237.7, 196.8), turned to 0 degrees
- moved C22 133.7 mm to (235.9, 191.8), turned to 90 degrees
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Connections:
- U5 pad 12: /GPIO5 -> /GPIO7
- U5 pad 14: /GPIO7 -> /GPIO5
Routing:
- net +3V3: track 9.37 -> 40.7 mm, vias 0 -> 7
- net +1V1: track 0.00 -> 15.1 mm, vias 0 -> 1
- net /USB_D+: track 5.55 -> 20.5 mm
- net /QSPI_SD2: track 0.00 -> 14.6 mm
- net /GPIO0: track 3.07 -> 17.6 mm, vias 0 -> 2
- net /GPIO2 SDA: track 0.00 -> 13.4 mm
- net /USB_D-: track 7.79 -> 21.0 mm
- net /QSPI_SD3: track 0.00 -> 12.1 mm
- net /GPIO3 SCL: track 0.00 -> 12.0 mm
- net /RUN: track 0.00 -> 11.9 mm
- net /XIN: track 0.00 -> 10.8 mm
- net /QSPI_SCLK: track 0.00 -> 10.7 mm
- net /GPIO25: track 0.00 -> 10.6 mm, vias 0 -> 2
- net /QSPI_SD0: track 0.00 -> 9.24 mm
- net GND: track 15.5 -> 24.1 mm, vias 2 -> 29
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- added copper zone on F.Cu, net +1V1
- added copper zone on F.Cu, net /VREG_LX
Other:
- board outline added: 35 x 55 mm
- board text added: "random bullshit put wherever tehres space"

Commit message: moar tracin
Parts:
- moved C27 391.2 mm to (188.8, 262.2)
- moved C36 391.2 mm to (206.8, 275.0)
- moved C38 391.2 mm to (204.8, 275.0)
- moved C40 391.2 mm to (203.8, 275.0)
- moved C46 391.2 mm to (273.0, 262.4)
- moved C47 391.2 mm to (274.3, 276.4)
- moved C48 391.2 mm to (281.9, 285.3)
- moved C51 391.2 mm to (298.4, 280.2)
- moved FB1 391.2 mm to (184.3, 262.7)
- moved J4 391.2 mm to (312.4, 276.4)
- moved L2 391.2 mm to (219.7, 275.1)
- moved L3 391.2 mm to (233.6, 270.0)
- moved L6 391.2 mm to (264.1, 271.3)
- moved L7 391.2 mm to (281.9, 276.4)
- moved R16 391.2 mm to (205.8, 275.0)
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- renumbered SW1 to RST, SW2 to RUN
Routing:
- net VBUS: track 23.8 -> 90.9 mm
- net /RUN: track 11.9 -> 58.1 mm, vias 0 -> 2
- net /SWCLK: track 0.00 -> 33.1 mm, vias 0 -> 2
- net /SWD: track 0.00 -> 32.3 mm, vias 0 -> 2
- net /QSPI_SS: track 0.13 -> 31.4 mm, vias 0 -> 2
- net /QSPI_SD1: track 0.00 -> 30.6 mm, vias 0 -> 2
- net /GPIO12: track 0.00 -> 23.1 mm, vias 0 -> 1
- net /GPIO29_ADC3: track 0.00 -> 21.8 mm, vias 0 -> 1
- net /GPIO13: track 0.00 -> 21.5 mm, vias 0 -> 1
- net /GPIO28_ADC2: track 0.00 -> 21.4 mm, vias 0 -> 1
- net /GPIO26_ADC0: track 0.00 -> 21.3 mm, vias 0 -> 1
- net /GPIO27_ADC1: track 0.00 -> 20.3 mm, vias 0 -> 1
- net /GPIO14: track 0.00 -> 20.0 mm, vias 0 -> 1
- net /GPIO15: track 0.00 -> 19.8 mm, vias 0 -> 1
- net /GPIO0: track 17.6 -> 35.6 mm, vias 2 -> 3
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- added copper zone on In2.Cu, net +3V3
- added copper zone on B.Cu, net GND
- added copper zone on F.Cu, net GND
- added copper zone on In1.Cu, net GND
Other:
- board size 35 x 55 mm -> 35.1 x 55 mm
- board text added: "radio pins"
- board text removed: "random bullshit put wherever tehres space"

Commit message: Fix most DRC errors and preliminary CC1200 fit
Parts:
- moved C3 291.6 mm to (253.1, 204.8), turned to -90 degrees
- moved C44 87.5 mm to (313.8, 217.9)
- moved L2 87.5 mm to (285.9, 217.9)
- moved C43 87.5 mm to (294.7, 217.9)
- moved L6 87.5 mm to (330.3, 214.1)
- moved C45 87.5 mm to (326.5, 230.6)
- moved C47 87.5 mm to (340.5, 219.2)
- moved C48 87.5 mm to (348.1, 228.1)
- moved C51 87.5 mm to (364.6, 223.0)
- moved J4 87.5 mm to (378.6, 219.2)
- moved L4 87.5 mm to (304.9, 217.9)
- moved L5 87.5 mm to (306.2, 230.6)
- moved L7 87.5 mm to (348.1, 219.2)
- moved L9 87.5 mm to (368.4, 219.2)
- moved C46 87.5 mm to (339.2, 205.2)
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- renumbered RST to BOOT
Routing:
- net GND: track 25.3 -> 8.50 mm, vias 32 -> 41
- net +3.3VA: track 21.2 -> 10.8 mm, vias 0 -> 13
- net +3V3: track 41.8 -> 48.0 mm, vias 17 -> 19
- net /GPIO23: track 4.13 -> 0.00 mm
- net /GPIO24: track 3.93 -> 0.00 mm
- net /GPIO21: track 3.85 -> 0.00 mm
- net /CC1200/TCXO_CLK: track 3.07 -> 6.43 mm
- net /GPIO9: track 0.00 -> 2.27 mm
- net /SWCLK: track 33.1 -> 30.9 mm, vias 2 -> 1
- net /GPIO22: track 0.00 -> 1.57 mm
- net /SWD: track 32.3 -> 30.8 mm, vias 2 -> 1
- net Net-(U7-DCPL_XOSC): track 2.40 -> 3.40 mm
- net Net-(U7-LPF0): track 2.77 -> 3.76 mm
- net Net-(U7-DCPL): track 2.56 -> 1.63 mm
- net VBUS: track 90.9 -> 90.4 mm
- added copper zone on F.Cu, net +3.3VA
- added copper zone on In2.Cu, net +3.3VA
Other:
- board text removed: "CC1200"
- board text removed: "Change 3.3VA traces that are next to eachother with copper pours Probably below RF section replace 3.3V layer with 3.3VA? Rethink components names silkscreen sizes, because they be pretty larg for this scale"

Commit message: random bullshit go
Parts:
- moved J4 118.5 mm to (260.0, 220.2)
Other:
- board text added: "20 19 18 17 16 15 14 13 12 G"
- board text added: "S S 29 28 27 26 RUN G 3v3 5V"
Changed lines of the file:
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@@
 	(footprint "Connector_Coaxial:U.FL_Hirose_U.FL-R-SMT-1_Vertical"
 		(layer "F.Cu")
-		(at 378.56 219.18)
+		(at 260.02 220.15)
 		(descr "Hirose U.FL Coaxial https://www.hirose.com/product/en/products/U.FL/U.FL-R-SMT-1%2810%29/")
 		(tags "Hirose U.FL Coaxial")
@@
 			(polygon
 				(pts
-					(xy 380.135 218.23) (xy 378.045 218.23) (xy 378.045 220.13) (xy 380.135 220.13)
+					(xy 261.595 219.2) (xy 259.505 219.2) (xy 259.505 221.1) (xy 261.595 221.1)
 				)
 			)
@@
 		(tags "Miniature Crystal Clock Oscillator TG2520 series SMD SMT")
 		(property "Reference" "Y2"
-			(at -1.1 2.35 180)
+			(at -1.925 0 180)
 			(layer "F.SilkS")
 			(effects
@@
 	)
 	(gr_line
-		(start 249.47 183.005)
-		(end 247.67 179.605)
+		(start 249.47 179.605)
+		(end 247.67 183.005)
 		(stroke
 			(width 0.12)
@@
 	)
 	(gr_line
-		(start 249.47 179.605)
-		(end 247.67 183.005)
+		(start 249.47 183.005)
+		(end 247.67 179.605)
 		(stroke
 			(width 0.12)
@@
 		(layer "F.SilkS")
 	)
-	(gr_line
-		(start 247.37 203.7)
-		(end 248.05 202.5)
+	(gr_rect
+		(start 39 37)
+		(end 459 334)
 		(stroke
-			(width 0.1)
+			(width 0.15)
 			(type default)
 		)
+		(fill no)
 		(layer "Dwgs.User")
 	)
@@
 		(layer "Dwgs.User")
 	)
-	(gr_rect
-		(start 39 37)
-		(end 459 334)
+	(gr_line
+		(start 247.37 203.7)
+		(end 248.05 202.5)
 		(stroke
-			(width 0.15)
+			(width 0.1)
 			(type default)
 		)
-		(fill no)
 		(layer "Dwgs.User")
 	)
 	(gr_arc
-		(start 262.75 169.15)
-		(mid 263.457107 169.442893)
-		(end 263.75 170.15)
-		(stroke
-			(width 0.2)
-			(type default)
-		)
-		(layer "Edge.Cuts")
-	)
-	(gr_arc
 		(start 228.7 170.15)
 		(mid 228.992893 169.442893)
@@
 	)
 	(gr_line
-		(start 229.7 169.15)
-		(end 262.75 169.15)
+		(start 228.7 223.15)
+		(end 228.7 170.15)
 		(stroke
 			(width 0.2)
@@
 		(layer "Edge.Cuts")
 	)
-	(gr_arc
-		(start 263.75 223.15)
-		(mid 263.457107 223.857107)
-		(end 262.75 224.15)
+	(gr_line
+		(start 229.7 169.15)
+		(end 262.75 169.15)
 		(stroke
 			(width 0.2)
@@
 		(layer "Edge.Cuts")
 	)
-	(gr_line
-		(start 228.7 223.15)
-		(end 228.7 170.15)
+	(gr_arc
+		(start 262.75 169.15)
+		(mid 263.457107 169.442893)
+		(end 263.75 170.15)
 		(stroke
 			(width 0.2)
@@
 		(layer "Edge.Cuts")
 	)
+	(gr_arc
+		(start 263.75 223.15)
+		(mid 263.457107 223.857107)
+		(end 262.75 224.15)
+		(stroke
+			(width 0.2)
+			(type default)
+		)
+		(layer "Edge.Cuts")
+	)
+	(gr_text "S\n\nS\n\n29\n\n28\n\n27\n\n26\n\nRUN\n\nG\n\n3v3\n\n5V"
+		(at 232.45 189.7 0)
+		(layer "F.SilkS")
+		(effects
+			(font
+				(size 0.79 0.79)
+				(thickness 0.1)
+			)
+			(justify left top)
+		)
+	)
+	(gr_text "20\n\n19\n\n18\n\n17\n\n16\n\n15\n\n14\n\n13\n\n12\n\nG"
+		(at 259.7 213.5 0)
+		(layer "F.SilkS")
+		(effects
+			(font
+				(size 0.79 0.79)
+				(thickness 0.1)
+			)
+			(justify right bottom)
+		)
+	)
 	(gr_text "radio\npins"

Commit message: RF section complete, I think
Parts:
- moved C50 119.7 mm to (241.1, 222.7), turned to 180 degrees
- moved L9 111.1 mm to (257.3, 218.3), turned to 0 degrees
- moved C51 109.0 mm to (255.7, 218.8), turned to -90 degrees
- moved L8 106.7 mm to (254.1, 218.3), turned to 0 degrees
- moved C49 105.4 mm to (245.4, 222.7)
- moved C46 96.9 mm to (243.8, 222.2), turned to 90 degrees
- moved L7 95.6 mm to (252.5, 220.3)
- moved C48 94.8 mm to (253.6, 220.3)
- moved R17 89.2 mm to (242.8, 222.2), turned to 90 degrees
- moved C47 87.9 mm to (252.6, 222.0), turned to 0 degrees
- moved L6 87.8 mm to (242.8, 220.1), turned to 90 degrees
- moved C45 75.5 mm to (252.0, 218.3), turned to 0 degrees
- moved C44 67.6 mm to (246.2, 216.6)
- moved L5 57.6 mm to (249.9, 218.3), turned to 0 degrees
- moved L4 57.3 mm to (247.6, 217.8)
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Routing:
- net /CC1200/PA: track 0.00 -> 12.1 mm
- net /CC1200/TRX_SW: track 0.00 -> 10.8 mm, vias 0 -> 2
- net /CC1200/LNA_N: track 0.00 -> 7.99 mm
- net /CC1200/LNA_P: track 0.00 -> 7.95 mm
- net +3V3: track 48.0 -> 43.7 mm, vias 19 -> 21
- net Net-(C45-Pad2): track 0.00 -> 3.65 mm
- net Net-(J4-In): track 0.00 -> 3.50 mm
- net +3.3VA: track 10.8 -> 14.1 mm, vias 13 -> 18
- net Net-(C43-Pad2): track 0.00 -> 3.06 mm
- net Net-(C47-Pad2): track 0.00 -> 2.93 mm
- net Net-(C51-Pad1): track 0.00 -> 2.23 mm
- net Net-(C46-Pad2): track 0.00 -> 2.13 mm
- net GND: vias 41 -> 48
- added copper zone on F.Cu, net +3V3

Commit message: Finished PCB???
Parts:
- moved C47 272.5 mm to (501.4, 333.2)
- moved C50 272.5 mm to (489.9, 333.9)
- moved C6 272.5 mm to (497.4, 298.2)
- moved J2 272.5 mm to (479.8, 324.2)
- moved L3 272.5 mm to (494.6, 329.5)
- moved L6 272.5 mm to (491.6, 331.3)
- moved R1 272.5 mm to (497.4, 292.5)
- moved R10 272.5 mm to (500.6, 307.0)
- moved R12 272.5 mm to (494.6, 303.5)
- moved R17 272.5 mm to (491.6, 333.4)
- moved R7 272.5 mm to (497.4, 296.0)
- moved R8 272.5 mm to (495.5, 318.8)
- moved U1 272.5 mm to (486.4, 295.8)
- moved Y2 272.5 mm to (485.6, 318.6)
- moved C1 272.5 mm to (493.6, 320.5)
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- renumbered BOOT to SW1, RUN to SW2
Connections:
- U7 pad 10: /GPIO22 -> /GPIO24
- U7 pad 2: /GPIO21 -> /GPIO22
- U7 pad 3: /GPIO24 -> /GPIO21
Routing:
- net /GPIO21: track 0.00 -> 40.2 mm, vias 0 -> 2
- net /GPIO24: track 0.00 -> 39.3 mm, vias 0 -> 2
- net /GPIO22: track 1.57 -> 40.0 mm, vias 0 -> 2
- net /GPIO23: track 0.00 -> 36.5 mm, vias 0 -> 2
- net /GPIO8: track 0.00 -> 29.1 mm
- net /GPIO10: track 0.00 -> 27.3 mm
- net /GPIO11: track 0.00 -> 26.4 mm
- net /GPIO9: track 2.27 -> 27.5 mm, vias 0 -> 2
- net +1V1: track 15.1 -> 30.7 mm, vias 1 -> 0
- net +3V3: track 43.7 -> 33.5 mm, vias 21 -> 26
- net /SWD: track 30.8 -> 35.3 mm
- net /GPIO26_ADC0: track 21.3 -> 25.4 mm
- net /GPIO27_ADC1: track 20.3 -> 24.2 mm
- net /SWCLK: track 30.9 -> 34.8 mm
- net /GPIO28_ADC2: track 21.4 -> 24.0 mm
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Other:
- board size 35.1 x 55 mm -> 35 x 55 mm
- board text added: "3V3"
- board text added: "BOOT"
- board text added: "GND"
- board text added: "GP12"
- board text added: "GP13"
- board text added: "GP14"
- board text added: "GP15"
- board text added: "GP16"
- board text added: "GP17"
- board text added: "GP18"
- board text added: "GP19"
- board text added: "GP20"
- board text added: "GP26"
- board text added: "GP27"
- board text added: "GP28"
- board text added: "GP29"
- board text added: "RESET"
- board text added: "RUN"
- board text added: "SWCLK"
- board text added: "SWDIO"
- board text added: "VBUS"
- board text removed: "20 19 18 17 16 15 14 13 12 G"
- board text removed: "Main Sheet"
- board text removed: "S S 29 28 27 26 RUN G 3v3 5V"
- board text removed: "radio pins"

Commit message: QoL changes
Routing:
- net GND: track 7.71 -> 4.00 mm
- net Net-(JP1-C): track 4.15 -> 2.59 mm
- net +3V3: track 33.5 -> 34.3 mm, vias 26 -> 27
Other:
- board text added: "0x76 (default)"
- board text added: "0x77"
- board text added: "BMP390 I2C address selector"
