File: CARP.kicad_pcb (KiCad board)
At the start: 4 copper layers, 35 x 55 mm, 95 parts, among them J1 USB_C_Receptacle_USB2.0_14P, J2 Conn_01x10, J3 Conn_01x10, J4 U.fl, SW1 SW_Push, SW2 SW_Push, U1 W25Q128JVSIMTR (16MB), U2 W25Q32RVXHJQ (2MB), U3 LM1117IMPX-3.3, U4 RP2350_60QFN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

Commit message: silkscreen
Parts:
- added REF**: Smolhaj_Scale_0.1, Symbol:Smolhaj_Scale_0.1, B.Cu at (489.2, 272.6)
Other:
- board text added: "(default) 0x76"
- board text added: "Aria Horak Marcin Czop"
- board text removed: "0x76 (default)"
