File: _autosave-_autosave-CARP.kicad_pcb (KiCad board)
At the start: 4 copper layers, 95 parts, among them J1 USB_C_Receptacle_USB2.0_14P, J2 Conn_01x10, J3 Conn_01x10, J4 U.fl, SW1 SW_Push, SW2 SW_Push, U1 W25Q128JVSIMTR (16MB), U2 W25Q32RVXHJQ (2MB), U3 LM1117IMPX-3.3, U4 RP2350_60QFN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

Commit message: further work on the essential modules
Parts:
- moved C3 219.5 mm to (282.6, 152.2), turned to 0 degrees
- moved J2 206.9 mm to (213.7, 199.7)
- moved J3 180.9 mm to (269.1, 222.9), turned to 180 degrees
- moved C2 171.6 mm to (243.5, 211.2), turned to 180 degrees
- moved R2 168.7 mm to (250.0, 239.8), turned to -90 degrees
- moved R1 168.0 mm to (250.0, 243.2), turned to -90 degrees
- moved C1 167.7 mm to (241.8, 213.6), turned to 90 degrees
- moved R7 167.4 mm to (250.0, 246.7), turned to 90 degrees
- moved C6 166.7 mm to (249.7, 249.0), turned to 0 degrees
- moved U2 161.8 mm to (245.7, 244.7), turned to -90 degrees
- moved Y1 156.2 mm to (244.5, 213.6), turned to 0 degrees
- moved R6 151.7 mm to (238.1, 241.5), turned to -90 degrees
- moved C5 148.4 mm to (236.5, 247.3), turned to -90 degrees
- moved R3 144.1 mm to (231.1, 234.0), turned to 0 degrees
- moved R8 141.5 mm to (245.5, 211.2), turned to 180 degrees
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Routing:
- net /XIN: track 0.00 -> 10.2 mm
- net GND: track 15.5 -> 22.9 mm, vias 2 -> 7
- net Net-(U4-USB_DP): track 0.00 -> 4.15 mm
- net Net-(U4-USB_DM): track 0.00 -> 3.84 mm
- net Net-(C2-Pad1): track 0.00 -> 2.87 mm
- net /VREG_AVDD: track 0.00 -> 2.85 mm
- net +3V3: track 9.37 -> 12.2 mm
- net +1V1: track 0.00 -> 2.54 mm, vias 0 -> 1
- net /XOUT: track 0.00 -> 2.34 mm
- added copper zone on F.Cu, net +1V1
- added copper zone on F.Cu, net /VREG_LX
Other:
- board text added: "1v1 deco"
- board text added: "3v3 deco"
- board text added: "random bullshit put wherever tehres space"
