File: CARP.kicad_sch (KiCad schematic)
At the start: 55 parts, among them J1 USB_C_Receptacle_USB2.0_14P, J2 Conn_01x10, J3 Conn_01x10, SW1 SW_Push, SW2 SW_Push, U1 W25Q128JVSIMTR (16MB), U2 W25Q32RVXHJQ (2MB), U3 LM1117IMPX-3.3, U4 RP2350_60QFN, U5 LSM6DSO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

Commit message: work
Parts:
- C23: footprint Capacitor_SMD:C_0402_1005Metric -> Capacitor_SMD:C_0603_1608Metric
- R14, R15: footprint PCM_Resistor_SMD_AKL:R_0603_1608Metric -> Resistor_SMD:R_0402_1005Metric
- SW2: footprint Button_Switch_SMD:SW_SPST_PTS645Sx43SMTR92 -> Button_Switch_SMD:SW_Push_1P1T_NO_Vertical_Wuerth_434133025816
Connections:
- net GPIO5: now also U5.14 (SDA); no longer U5.12 (CS)
- net GPIO7: now also U5.12 (CS); no longer U5.14 (SDA)
Changed lines of the file:
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@@
 		)
 	)
-	(label "GPIO5"
-		(at 386.08 224.79 180)
-		(effects
-			(font
-				(size 1.27 1.27)
-			)
-			(justify right bottom)
-		)
-	)
 	(label "QSPI_SD0"
 		(at 162.56 147.32 0)
@@
 		)
 	)
+	(label "GPIO5"
+		(at 386.08 219.71 180)
+		(effects
+			(font
+				(size 1.27 1.27)
+			)
+			(justify right bottom)
+		)
+	)
 	(label "GPIO11"
 		(at 255.27 160.02 180)
@@
 		)
 	)
+	(label "GPIO7"
+		(at 386.08 224.79 180)
+		(effects
+			(font
+				(size 1.27 1.27)
+			)
+			(justify right bottom)
+		)
+	)
 	(label "SWCLK"
 		(at 345.44 91.44 0)
@@
 		)
 	)
-	(label "GPIO7"
-		(at 386.08 219.71 180)
-		(effects
-			(font
-				(size 1.27 1.27)
-			)
-			(justify right bottom)
-		)
-	)
 	(label "GPIO2 SDA"
 		(at 255.27 137.16 180)
@@
 			)
 		)
-		(property "Footprint" "Button_Switch_SMD:SW_SPST_PTS645Sx43SMTR92"
+		(property "Footprint" "Button_Switch_SMD:SW_Push_1P1T_NO_Vertical_Wuerth_434133025816"
 			(at 153.67 172.72 0)
 			(effects
@@
 			)
 		)
-		(property "Footprint" "Capacitor_SMD:C_0402_1005Metric"
+		(property "Footprint" "Capacitor_SMD:C_0603_1608Metric"
 			(at 335.28 129.8448 0)
 			(effects
@@
 			)
 		)
-		(property "Footprint" "PCM_Resistor_SMD_AKL:R_0603_1608Metric"
+		(property "Footprint" "Resistor_SMD:R_0402_1005Metric"
 			(at 314.198 83.82 90)
 			(effects
@@
 			)
 		)
-		(property "Footprint" "PCM_Resistor_SMD_AKL:R_0603_1608Metric"
+		(property "Footprint" "Resistor_SMD:R_0402_1005Metric"
 			(at 315.722 83.82 90)
 			(effects

Commit message: Finished PCB???
Changed lines of the file:
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@@
 	(wire
 		(pts
+			(xy 355.6 147.32) (xy 368.3 147.32)
+		)
+		(stroke
+			(width 0)
+			(type default)
+		)
+	)
+	(wire
+		(pts
 			(xy 382.27 93.98) (xy 393.7 93.98)
 		)
@@
 	(wire
 		(pts
+			(xy 355.6 139.7) (xy 368.3 139.7)
+		)
+		(stroke
+			(width 0)
+			(type default)
+		)
+	)
+	(wire
+		(pts
 			(xy 153.67 95.25) (xy 153.67 97.79)
 		)
@@
 	(wire
 		(pts
-			(xy 355.6 134.62) (xy 368.3 134.62)
-		)
-		(stroke
-			(width 0)
-			(type default)
-		)
-	)
-	(wire
-		(pts
 			(xy 325.12 232.41) (xy 327.66 232.41)
 		)
@@
 	(wire
 		(pts
-			(xy 355.6 147.32) (xy 368.3 147.32)
-		)
-		(stroke
-			(width 0)
-			(type default)
-		)
-	)
-	(wire
-		(pts
 			(xy 386.08 219.71) (xy 378.46 219.71)
 		)
@@
 	(wire
 		(pts
+			(xy 355.6 134.62) (xy 368.3 134.62)
+		)
+		(stroke
+			(width 0)
+			(type default)
+		)
+	)
+	(wire
+		(pts
 			(xy 264.16 96.52) (xy 275.59 96.52)
 		)
@@
 	(wire
 		(pts
-			(xy 355.6 139.7) (xy 368.3 139.7)
-		)
-		(stroke
-			(width 0)
-			(type default)
-		)
-	)
-	(wire
-		(pts
 			(xy 43.18 36.83) (xy 44.45 36.83)
 		)
@@
 	(wire
 		(pts
-			(xy 355.6 137.16) (xy 368.3 137.16)
-		)
-		(stroke
-			(width 0)
-			(type default)
-		)
-	)
-	(wire
-		(pts
 			(xy 173.99 125.73) (xy 176.53 125.73)
 		)
@@
 	(wire
 		(pts
+			(xy 355.6 137.16) (xy 368.3 137.16)
+		)
+		(stroke
+			(width 0)
+			(type default)
+		)
+	)
+	(wire
+		(pts
 			(xy 275.59 86.36) (xy 275.59 85.09)
 		)
@@
 		)
 	)
-	(label "GPIO22"
-		(at 355.6 134.62 0)
-		(effects
-			(font
-				(size 1.27 1.27)
-			)
-			(justify left bottom)
-		)
-	)
 	(label "GPIO5"
 		(at 255.27 144.78 180)
@@
 		)
 	)
+	(label "GPIO21"
+		(at 355.6 139.7 0)
+		(effects
+			(font
+				(size 1.27 1.27)
+			)
+			(justify left bottom)
+		)
+	)
 	(label "GPIO20"
 		(at 393.7 93.98 180)
@@
 		)
 	)
-	(label "GPIO21"
-		(at 355.6 147.32 0)
-		(effects
-			(font
-				(size 1.27 1.27)
-			)
-			(justify left bottom)
-		)
-	)
 	(label "GPIO0"
 		(at 255.27 132.08 180)
@@
 		)
 	)
+	(label "GPIO24"
+		(at 355.6 134.62 0)
+		(effects
+			(font
+				(size 1.27 1.27)
+			)
+			(justify left bottom)
+		)
+	)
 	(label "VBUS"
 		(at 59.69 24.13 0)
@@
 		)
 	)
+	(label "GPIO22"
+		(at 355.6 147.32 0)
+		(effects
+			(font
+				(size 1.27 1.27)
+			)
+			(justify left bottom)
+		)
+	)
 	(label "GPIO3 SCL"
 		(at 255.27 139.7 180)
@@
 		)
 	)
-	(label "GPIO23"
-		(at 355.6 137.16 0)
-		(effects
-			(font
-				(size 1.27 1.27)
-			)
-			(justify left bottom)
-		)
-	)
 	(label "GPIO29_ADC3"
 		(at 255.27 208.28 180)
@@
 		)
 	)
+	(label "GPIO23"
+		(at 355.6 137.16 0)
+		(effects
+			(font
+				(size 1.27 1.27)
+			)
+			(justify left bottom)
+		)
+	)
 	(label "QSPI_SD1"
 		(at 95.885 163.195 180)
@@
 		(effects
 			(font
-				(size 1.27 1.27)
-			)
-			(justify left bottom)
-		)
-	)
-	(label "GPIO24"
-		(at 355.6 139.7 0)
-		(effects
-			(font

Commit message: QoL changes
Other:
- note added: "Default address: 0x76 Alternative address: 0x77"
Changed lines of the file:
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@@
+		)
+	)
+	(text "Default address: 0x76\nAlternative address: 0x77"
+		(exclude_from_sim no)
+		(at 297.688 190.5 0)
+		(effects
+			(font
+				(size 1.27 1.27)
+			)
 		)
 	)
